File: Keyboard.kicad_pcb (KiCad board)
At the start: 2 copper layers, 285.7 x 95.2 mm, 128 parts, among them SW1 MX_SW_solder, SW10 MX_SW_solder, SW11 MX_SW_solder, SW12 MX_SW_solder, SW13 MX_SW_solder, SW14 MX_SW_solder, SW15 MX_SW_solder, SW16 MX_SW_solder, SW17 MX_SW_solder, SW18 MX_SW_solder, SW19 MX_SW_solder, SW2 MX_SW_solder, SW20 MX_SW_solder, SW21 MX_SW_solder, SW22 MX_SW_solder, SW23 MX_SW_solder, SW24 MX_SW_solder, SW25 MX_SW_solder, SW26 MX_SW_solder, SW27 MX_SW_solder, SW28 MX_SW_solder, SW29 MX_SW_solder, SW3 MX_SW_solder, SW30 MX_SW_solder, SW31 MX_SW_solder, SW32 MX_SW_solder, SW33 MX_SW_solder, SW34 MX_SW_solder, SW35 MX_SW_solder, SW36 MX_SW_solder, SW37 MX_SW_solder, SW38 MX_SW_solder, SW39 MX_SW_solder, SW4 MX_SW_solder, SW40 MX_SW_solder, SW41 MX_SW_solder, SW42 MX_SW_solder, SW43 MX_SW_solder, SW44 MX_SW_solder, SW45 MX_SW_solder, SW46 MX_SW_solder, SW47 MX_SW_solder, SW48 MX_SW_solder, SW49 MX_SW_solder, SW5 MX_SW_solder, SW50 MX_SW_solder, SW51 MX_SW_solder, SW52 MX_SW_solder, SW53 MX_SW_solder, SW54 MX_SW_solder, SW55 MX_SW_solder, SW56 MX_SW_solder, SW57 MX_SW_solder, SW58 MX_SW_solder, SW59 MX_SW_solder, SW6 MX_SW_solder, SW60 MX_SW_solder, SW61 MX_SW_solder, SW7 MX_SW_solder, SW8 MX_SW_solder, SW9 MX_SW_solder, U1 Pico

Commit message: rerouted with correct pico placement
Parts:
- moved U1 0.13 mm to (41.4, 26.2)
Routing:
- net Row1: track 426.2 -> 264.1 mm, vias 1 -> 0
- net Row2: track 436.2 -> 287.4 mm
- net Row4: track 354.5 -> 298.6 mm
- net Row3: track 346.3 -> 290.6 mm
- net Col4: track 160.9 -> 193.9 mm
- net Col12: track 282.4 -> 276.3 mm
- net Col11: track 260.3 -> 265.3 mm
- net Col9: track 222.3 -> 227.1 mm
- net Col8: track 179.9 -> 184.4 mm
- net Col7: track 163.3 -> 167.9 mm
- net Col10: track 239.7 -> 244.2 mm
- net Col5: track 132.6 -> 130.2 mm
- net Col2: track 111.7 -> 109.7 mm
- net Col13: track 245.8 -> 244.0 mm
- net Col6: track 146.6 -> 147.3 mm
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Other:
- board size 285.7 x 95.2 mm -> 285.7 x 97.2 mm

Commit message: removed errors
Routing:
- net Col3: track 136.9 -> 138.7 mm
- net Row3: track 290.6 -> 292.3 mm
- net Row5: track 345.0 -> 346.3 mm
- net Row4: track 298.6 -> 299.9 mm
- net Col2: track 109.7 -> 110.4 mm

Commit message: Export v1 .grb
Parts:
- moved SW40 70.9 mm to (307.8, 103.5)
- moved D13 70.9 mm to (309.4, 70.2)
- moved D14 70.9 mm to (338.0, 70.2)
- moved D20 70.9 mm to (185.6, 89.2)
- moved D22 70.9 mm to (223.7, 89.2)
- moved D24 70.9 mm to (261.8, 89.2)
- moved D27 70.9 mm to (318.9, 89.2)
- moved D32 70.9 mm to (152.2, 108.3)
- moved D34 70.9 mm to (190.3, 108.3)
- moved D36 70.9 mm to (228.4, 108.3)
- moved D37 70.9 mm to (247.5, 108.3)
- moved D39 70.9 mm to (285.6, 108.3)
- moved D4 70.9 mm to (137.9, 70.2)
- moved D40 70.9 mm to (304.6, 108.3)
- moved D47 70.9 mm to (199.8, 127.3)
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Other:
- board size 285.7 x 97.2 mm -> 285.7 x 97 mm

Commit message: Added mounting holes and generated .gbr's
Parts:
- added M1: MountingHole_3.2mm_M3, MountingHole:MountingHole_3.2mm_M3, F.Cu at (104.0, 104.0)
- added M2: MountingHole_3.2mm_M3, MountingHole:MountingHole_3.2mm_M3, F.Cu at (174.6, 142.9)
- added M3: MountingHole_3.2mm_M3, MountingHole:MountingHole_3.2mm_M3, F.Cu at (319.1, 104.0)
Connections:
- U1 pad 13: unconnected-(U1-Pad13) -> GND
- U1 pad 18: unconnected-(U1-Pad18) -> GND
- U1 pad 23: unconnected-(U1-Pad23) -> GND
- U1 pad 25: Col15 -> unconnected-(U1-Pad25)
- U1 pad 28: unconnected-(U1-Pad28) -> GND
- U1 pad 3: unconnected-(U1-Pad3) -> GND
- U1 pad 38: unconnected-(U1-Pad38) -> GND
- U1 pad 8: unconnected-(U1-Pad8) -> GND
Routing:
- net GND: track 0.00 -> 13.9 mm
- added copper zone on B.Cu, net GND
- added copper zone on F.Cu, net GND
Other:
- board text added: "60% Keyboard V1 Clemens Retra Nov 2022 github.com/EpicKiwiProCoder /Mechanical-Keyboard-Pcb"
